Commit message: add controller

File: mini_pupper_description/urdf/mini_pupper_description.urdf (robot description, URDF)
Before this commit: robot mini_pupper_description, 17 links, 16 joints
Links:
- added link base_dummy
Joints:
- added joint dummy_joint: type fixed, parent base_dummy, child base_link

Commit message: fix urdf

File: mini_pupper_description/urdf/mini_pupper_description.urdf (robot description, URDF)
Before this commit: robot mini_pupper_description, 18 links, 17 joints
Joints:
- joint base_lb1: limit lower=-3.14 upper=3.14 effort=0 velocity=0 -> lower=-3.14 upper=3.14 effort=3.0 velocity=1.0
- joint base_lf1: limit lower=-3.14 upper=3.14 effort=0 velocity=0 -> lower=-3.14 upper=3.14 effort=3.0 velocity=1.0
- joint base_rb1: limit lower=-3.14 upper=3.14 effort=0 velocity=0 -> lower=-3.14 upper=3.14 effort=3.0 velocity=1.0
- joint base_rf1: limit lower=-3.14 upper=3.14 effort=0 velocity=0 -> lower=-3.14 upper=3.14 effort=3.0 velocity=1.0
- joint lb1_lb2: limit lower=-3.14 upper=3.14 effort=0 velocity=0 -> lower=-3.14 upper=3.14 effort=3.0 velocity=1.0
- joint lb2_lb3: limit lower=-3.14 upper=3.14 effort=0 velocity=0 -> lower=-3.14 upper=3.14 effort=3.0 velocity=1.0
- joint lf1_lf2: limit lower=-3.14 upper=3.14 effort=0 velocity=0 -> lower=-3.14 upper=3.14 effort=3.0 velocity=1.0
- joint lf2_lf3: limit lower=-3.14 upper=3.14 effort=0 velocity=0 -> lower=-3.14 upper=3.14 effort=3.0 velocity=1.0
- joint rb1_rb2: limit lower=-3.14 upper=3.14 effort=0 velocity=0 -> lower=-3.14 upper=3.14 effort=3.0 velocity=1.0
- joint rb2_rb3: limit lower=-3.14 upper=3.14 effort=0 velocity=0 -> lower=-3.14 upper=3.14 effort=3.0 velocity=1.0
- joint rf1_rf2: limit lower=-3.14 upper=3.14 effort=0 velocity=0 -> lower=-3.14 upper=3.14 effort=3.0 velocity=1.0
- joint rf2_rf3: limit lower=-3.14 upper=3.14 effort=0 velocity=0 -> lower=-3.14 upper=3.14 effort=3.0 velocity=1.0

Commit message: fix urdf

File: mini_pupper_description/urdf/mini_pupper_description.urdf (robot description, URDF)
Before this commit: robot mini_pupper_description, 18 links, 17 joints
Joints:
- joint base_lb1: limit lower=-3.14 upper=3.14 effort=3.0 velocity=1.0 -> lower=-3.14 upper=3.14 effort=10.0 velocity=10.0
- joint base_lf1: limit lower=-3.14 upper=3.14 effort=3.0 velocity=1.0 -> lower=-3.14 upper=3.14 effort=10.0 velocity=10.0
- joint base_rb1: limit lower=-3.14 upper=3.14 effort=3.0 velocity=1.0 -> lower=-3.14 upper=3.14 effort=10.0 velocity=10.0
- joint base_rf1: limit lower=-3.14 upper=3.14 effort=3.0 velocity=1.0 -> lower=-3.14 upper=3.14 effort=10.0 velocity=10.0
- joint lb1_lb2: limit lower=-3.14 upper=3.14 effort=3.0 velocity=1.0 -> lower=-3.14 upper=3.14 effort=10.0 velocity=10.0
- joint lb2_lb3: limit lower=-3.14 upper=3.14 effort=3.0 velocity=1.0 -> lower=-3.14 upper=3.14 effort=10.0 velocity=10.0
- joint lf1_lf2: limit lower=-3.14 upper=3.14 effort=3.0 velocity=1.0 -> lower=-3.14 upper=3.14 effort=10.0 velocity=10.0
- joint lf2_lf3: limit lower=-3.14 upper=3.14 effort=3.0 velocity=1.0 -> lower=-3.14 upper=3.14 effort=10.0 velocity=10.0
- joint rb1_rb2: limit lower=-3.14 upper=3.14 effort=3.0 velocity=1.0 -> lower=-3.14 upper=3.14 effort=10.0 velocity=10.0
- joint rb2_rb3: limit lower=-3.14 upper=3.14 effort=3.0 velocity=1.0 -> lower=-3.14 upper=3.14 effort=10.0 velocity=10.0
- joint rf1_rf2: limit lower=-3.14 upper=3.14 effort=3.0 velocity=1.0 -> lower=-3.14 upper=3.14 effort=10.0 velocity=10.0
- joint rf2_rf3: limit lower=-3.14 upper=3.14 effort=3.0 velocity=1.0 -> lower=-3.14 upper=3.14 effort=10.0 velocity=10.0
